File: Hardware/board.brd (EAGLE design)
At the start: 46 x 35 mm, 105 parts, among them IC1 BQ25180YBGR, IC2 DRV2605YZFR, IC3 BMA421, IC9 RT6160AWSC, J1 503480-2400, J2 TC2030-IDC, J4 KH-TYPE-C-16P, Q1 20V/4.2A/52mΩ/1.4W, Q3 SI1308EDL-T1-GE3, U1 NRF52840_QF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

Commit message: Update board.brd
Parts:
- L1: device InkTime_v5:NORDIC_NRF_2_RESC0402_M -> InkTime_v5:NORDIC_NRF_2_RESC0402_L
- moved X2 39.6 mm to (8.63, 14.9)
- moved TP_BAT_GND 34.5 mm to (-18.5, -13.0)
- moved TP_GND 29.6 mm to (-19.7, -9.40)
- moved TP_SWDIO 28.3 mm to (-5.10, -14.6)
- moved X1 28.3 mm to (-7.90, 2.22)
- moved TP_SWO 24.8 mm to (10.3, 3.53)
- moved C9 23.6 mm to (-0.20, 5.00)
- moved IC3 23.1 mm to (3.05, -6.64), turned to 270 degrees
- moved C13 22.9 mm to (-2.70, 3.40)
- moved IC1 22.2 mm to (11.8, -6.70)
- moved C5 22.0 mm to (-2.50, 7.90)
- moved C11 20.8 mm to (12.4, 6.10)
- moved C6 20.3 mm to (2.40, -12.5)
- moved R9 19.1 mm to (-5.30, 3.10), turned to 90 degrees
- moved TP_RESET 19.0 mm to (-4.35, -4.02)
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Connections:
- removed net SCL/2.4C: U1.P$M2
- removed net SDA/2.4C: U1.P$L1
- removed net VBAT/1.2A: TP_VBAT.TP
- net SCL: now also U1.P$M2
- net SDA: now also U1.P$L1
- net VBAT: now also TP_VBAT.TP
Routing:
- net GND: track 363.6 -> 15.4 mm, vias 7 -> 53
- net N$18: track 98.5 -> 33.2 mm, vias 9 -> 3
- net N$19: track 2.04 -> 43.8 mm, vias 0 -> 2
- net 3V3: track 176.9 -> 136.3 mm, vias 16 -> 7
- net HAPTIC_EN: track 49.4 -> 9.08 mm, vias 6 -> 2
- net EPD_RST: track 0.00 -> 40.2 mm, vias 0 -> 6
- net N$9: track 49.9 -> 10.2 mm, vias 3 -> 0
- net P0.14: track 55.7 -> 21.1 mm
- net EPD_CS: track 0.00 -> 31.2 mm, vias 0 -> 4
- net SDA: track 41.4 -> 70.8 mm
- net N$13: track 32.7 -> 4.95 mm
- net N$1: track 3.40 -> 30.2 mm, vias 0 -> 3
- net SWDCLK: track 24.9 -> 48.8 mm, vias 6 -> 2
- net N$8: track 45.7 -> 22.1 mm, vias 5 -> 3
- net N$3: track 45.6 -> 22.1 mm, vias 9 -> 3
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- added copper zone on layer 1, net GND
- added copper zone on layer 16, net GND
- added copper zone on layer 2, net GND
