File: Hardware/schematic.sch (EAGLE design)
At the start: 57 parts, among them IC1 BQ25180YBGR, IC3 BMA421, IC9 RT6160AWSC, J1 TC2030-IDC, U1 NRF52840_QF, X1 32MHz, X2 32.768KHz

Commit message: Update schematic.sch
Parts:
- removed R1: 10K, InkTime_v5:CPF0201D7K68C1_CPF0201D7K68C1
- added C1-EP-DR: 10uF, InkTime_v5:NORDIC_NRF_3_CAPACITOR_0402_L
- added C2-EP-DR: 4.7uF/25V, InkTime_v5:NORDIC_NRF_3_CAPACITOR_0402_L
- added C27, C34, C42: 0.1uF, InkTime_v5:GRM011R60J152KE01L_2_GRM011R60J152KE01L
- added C29, C30, C31, C32: 1uF, InkTime_v5:GRM011R60J152KE01L_2_GRM011R60J152KE01L
- added C43: 4.7uF, InkTime_v5:NORDIC_NRF_3_CAPACITOR_0402_L
- added D2, D5, DE_PUS: MBR0530, InkTime_v5:ESP32_C6_LIBRARY_5_MBR0530
- added D3: USBLC6-2SC6Y, InkTime_v5:ESP32_C6_LIBRARY_3_USBLC6-2SC6Y
- added EPD_C1, EPD_C10, EPD_C11, EPD_C12, EPD_C2, EPD_C6, EPD_C7, EPD_C8, EPD_C9: 1uF/50V, InkTime_v5:NORDIC_NRF_3_CAPACITOR_0402_L
- added EPD_C5: 0.1uF/50V, InkTime_v5:NORDIC_NRF_3_CAPACITOR_0402_L
- added IC2: DRV2605YZFR, InkTime_v5:DRV2605YZFR_DRV2605YZFR
- added J2: TC2030-IDC, InkTime_v5:TC2030-IDC_TC2030-IDC
- added J4: KH-TYPE-C-16P, InkTime_v5:KH-TYPE-C-16P_KH-TYPE-C-16P
- added L5: 68uH, InkTime_v5:ESP32_C6_LIBRARY_2_744043680IND_4828-WE-TPC_WRE
- added Q1: 20V/4.2A/52mΩ/1.4W, InkTime_v5:ESP32_C6_LIBRARY_4_ESP32_WROVER_SPARKFUN-DISCRETESEMI_MOSFET_PCH-DMG2305UX-7
- added Q3: SI1308EDL-T1-GE3, InkTime_v5:ESP32_C6_LIBRARY_6_SI1308EDL-T1-GE3
- added R1_EP_DR: 0.47, InkTime_v5:CPF0201D7K68C1_CPF0201D7K68C1
- added R1_USB, R2_USB: 5K1, InkTime_v5:CPF0201D7K68C1_CPF0201D7K68C1
- added R2_EP_DR, R9, R_PWR_EPD: 10K, InkTime_v5:CPF0201D7K68C1_CPF0201D7K68C1
- added R5, R7, R8: 10k, InkTime_v5:CPF0201D7K68C1_CPF0201D7K68C1
- added R_TYPE_SEL: 2.2, InkTime_v5:CPF0201D7K68C1_CPF0201D7K68C1
- added SJ1: 0, InkTime_v5:ESP32_C6_LIBRARY_7_JUMPER_SJ
- added SW_DN, SW_ENT, SW_UP: 2025-10-22_07-23-44_LIBRARY_EVP-AKE31ASW_EVP-AKE31A_PAN, InkTime_v5:2025-10-22_07-23-44_LIBRARY_EVP-AKE31ASW_EVP-AKE31A_PAN
- added TP_BAT_GND, TP_ON, TP_OP, TP_VBAT: HECTOR_WATCH_1_TPTP20R, InkTime_v5:HECTOR_WATCH_1_TPTP20R
- added U3: ESP32_C6_LIBRARY_MAX17048G+T10, InkTime_v5:ESP32_C6_LIBRARY_MAX17048G+T10
- C1, C10, C11, C12, C13, C16, C17, C18, C19, C2, C22, C3, C4, C5, C7, C8, C9: device InkTime_v5:NORDIC_NRF_3_CAPACITOR_0402_M -> InkTime_v5:NORDIC_NRF_3_CAPACITOR_0201_L
- C14, C15, C20, C21, C25, C33, C39, C6: device InkTime_v5:NORDIC_NRF_3_CAPACITOR_0402_M -> InkTime_v5:NORDIC_NRF_3_CAPACITOR_0402_L
- C24: device InkTime_v5:NORDIC_NRF_3_CAPACITOR_0201_M -> InkTime_v5:NORDIC_NRF_3_CAPACITOR_0402_L
- J1: value TC2030-IDC -> 503480-2400; device InkTime_v5:TC2030-IDC_TC2030-IDC -> InkTime_v5:503480-2400_503480-2400
- L2: device InkTime_v5:NORDIC_NRF_2_INDUCTOR_0402_M -> InkTime_v5:NORDIC_NRF_2_INDUCTOR_0603_L
- L3: value 15uH -> 15nH; device InkTime_v5:NORDIC_NRF_2_INDUCTOR_0402_M -> InkTime_v5:NORDIC_NRF_2_INDUCTOR_0201_L
Connections:
- new net DN: D3.I/O1_1, J4.DN1, J4.DN2
- new net DP: D3.I/O2_1, J4.DP1, J4.DP2
- new net EPD_3V3: C1-EP-DR.1, EPD_C5.2, J1.15, J1.16, L5.2, Q1.D
- new net GDR: J1.2, Q3.G, R2_EP_DR.2
- new net N$12: R1_EP_DR.1, R_TYPE_SEL.2, SJ1.2
- new net N$16: C32.2, IC2.REG
- new net N$21: C2-EP-DR.1, D2.K, DE_PUS.A
- new net N$24: C2-EP-DR.2, D5.A, L5.1, Q3.D
- new net N$25: EPD_C2.2, J1.4
- new net N$26: EPD_C1.2, J1.5
- new net N$27: J4.CC2, R2_USB.1
- new net N$28: EPD_C7.2, J1.19
- new net N$30: EPD_C12.2, J1.24
- new net N$31: EPD_C6.2, J1.18
- new net N$32: EPD_C8.2, J1.20
- new net N$34: EPD_C10.2, J1.22
- new net N$36: J4.CC1, R1_USB.2
- new net OUT+: IC2.OUT+, TP_OP.TP
- new net OUT-: IC2.OUT-, TP_ON.TP
- new net PREVGH: D5.K, EPD_C9.2, J1.21
- new net PREVGL: D2.A, EPD_C11.2, J1.23
- new net RESE: J1.3, Q3.S, R1_EP_DR.2
- new net VBAT/1.2A: TP_VBAT.TP
- net 3V3: now also C34.2, IC2.VDD, J2.1, Q1.S, R5.2, R7.2, R8.2, R_PWR_EPD.2; no longer J1.1
- net ALERT: now also U3.!ALERT
- net D+: now also D3.I/O2_2
- net D-: now also D3.I/O1_2
- net EPD_BUSY: now also J1.9
- net EPD_CS: now also J1.12
- net EPD_DC: now also J1.11
- net EPD_RST: now also J1.10
- net GND: now also C1-EP-DR.2, C27.1, C29.1, C30.1, C31.1, C32.1, C34.1, C42.2, C43.2, D3.GND, DE_PUS.K, EPD_C1.1, EPD_C10.1, EPD_C11.1, EPD_C12.1, EPD_C2.1, EPD_C5.1, EPD_C6.1, EPD_C7.1, EPD_C8.1, EPD_C9.1, IC2.GND, IC2.IN/TRIG, J1.17, J1.8, J1.MP1, J1.MP2, J2.3, J2.5, J4.GND, J4.SHIELD, R1_USB.1, R2_EP_DR.1, R2_USB.2, R9.1, R_TYPE_SEL.1, SJ1.1, SW_DN.1, SW_ENT.1, SW_UP.1, TP_BAT_GND.TP, U3.CTG, U3.EP, U3.GND, U3.QSTRT; no longer J1.3, J1.5, R1.1
- net HAPTIC_EN: now also IC2.EN
- net MOSI: now also J1.14
- net N$1: now also R9.2; no longer R1.2
- net P0.13: now also C30.2, R5.1, SW_UP.2
- net P0.14: now also C31.2, R8.1, SW_ENT.2
- net P1.01: now also Q1.G, R_PWR_EPD.1
- net P1.02: now also C29.2, R7.1, SW_DN.2
- net RESET: now also J2.6; no longer J1.6
- net SCK: now also J1.13
- net SCL: now also IC2.SCL, U3.SCL
- net SDA: now also IC2.SDA, U3.SDA
- net SWDCLK: now also J2.4; no longer J1.4
- net SWDIO: now also J2.2; no longer J1.2
- net VBAT: now also C27.2, U3.CELL, U3.VDD
- net VBUS: now also C42.1, C43.1, D3.VBUS, J4.VBUS
Other:
- note added: "Buttons"
- note added: "DMG2305UX-7"
- note added: "E-Paper Display Connector"
- note added: "E-Paper Drive Circuit"
- note added: "Fuel Gauge"
- note added: "Haptic Driver"
- note added: "USB C Connector & ESD Protection"

Commit message: Update schematic.sch
Parts:
- L1: device InkTime_v5:NORDIC_NRF_2_INDUCTOR_0402_M -> InkTime_v5:NORDIC_NRF_2_INDUCTOR_0402_L
Connections:
- removed net SCL/2.4C: U1.P0.07@M2
- removed net SDA/2.4C: U1.P0.06@L1
- removed net VBAT/1.2A: TP_VBAT.TP
- net SCL: now also U1.P0.07@M2
- net SDA: now also U1.P0.06@L1
- net VBAT: now also TP_VBAT.TP
